File: 009pcb/009pcb4_12mil.brd (EAGLE design)
At the start: 50.8 x 45.7 mm, 26 parts, among them Q1 600mA/30V, Q2 600mA/30V, U1 V_REG_317SINK

Commit message: 009pcb6 and eagle libraries
Parts:
- moved BUZZER_1 2.84 mm to (36.8, 40.6)
- moved BUZZER_2 2.84 mm to (39.4, 40.6)
- moved CHARGER_HOLES 2.84 mm to (39.4, 35.6)
- moved LED_WHITE_ANODE 2.84 mm to (36.8, 38.1)
- moved LED_WHITE_CATHODE 2.84 mm to (39.4, 38.1)
- moved 5V_BOOSTER 2.84 mm to (50.8, 27.9)
- moved BOOSTER_25V 2.84 mm to (49.5, 24.1)
- moved CHARGER_BOARD 1.80 mm to (38.1, 8.89)
- moved R6 1.80 mm to (3.81, 38.1)
- moved HALL_EFFECT_SENSOR_HOLES 1.80 mm to (29.2, 40.6)
- moved R1 1.80 mm to (21.6, 35.6)
- moved R2 1.80 mm to (21.6, 38.1)
- moved R5 1.80 mm to (21.6, 33.0)
- moved R7 1.80 mm to (6.35, 38.1)
- moved R8 1.80 mm to (21.6, 40.6)
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Routing:
- net VOUT_BOOSTER: track 48.1 -> 88.1 mm, vias 0 -> 3
- net COLLECTOR: track 38.5 -> 58.9 mm, vias 0 -> 2
- net SCL: track 59.8 -> 40.0 mm
- net EN: track 16.6 -> 31.8 mm, vias 0 -> 2
- net 5V: track 21.2 -> 33.2 mm
- net GND: track 143.6 -> 155.2 mm
- net ADJUST: track 28.9 -> 35.1 mm, vias 0 -> 2
- net N$6: track 17.6 -> 14.1 mm
- net 3V: track 41.7 -> 44.9 mm, vias 0 -> 2
- net SDA: track 31.2 -> 28.4 mm
- net A0: track 17.7 -> 20.4 mm, vias 0 -> 2
- net BAT: track 24.3 -> 26.9 mm
- net VOUT_LM317: track 32.5 -> 30.4 mm
- net BASE: track 39.4 -> 40.8 mm, vias 0 -> 2
- net 5V_CHARGER: track 19.1 -> 19.2 mm, vias 0 -> 2
Other:
- board size 50.8 x 45.7 mm -> 55.9 x 48.3 mm
