File: 009pcb/009pcb6.sch (EAGLE design)
At the start: 27 parts

Commit message: 009pcb6.brd
Parts:
- removed ACTIVE_BUZZER, BATTERY, CHARGER_PORT, WHITE_LED: (no value), SparkFun-Connectors:CONN_02
- removed R8: 1 kΩ, RC0805JR-0720KL:RC0805JR-0720KL
- removed TRANSISTOR1: MMBT2222A-7-F, MMBT2222A-7-F:MMBT2222A-7-F
- added ACTIVE_BUZZER1, ACTIVE_BUZZER2, BATTERY1, BATTERY2, CHARGER_PORT1, CHARGER_PORT2, WHITE_LED1, WHITE_LED2: WIREPADSMD1,27-254, wirepad:WIREPADSMD1,27-254
- added C5, C6: GRT21BR61H475ME13L, GRT21BR61H475ME13L:GRT21BR61H475ME13L
- added INVERTER: BU4SU69G2-TR, BU4SU69G2-TR:BU4SU69G2-TR
- added L1: 2.2 uH, 74438357022:74438357022
- added R1_1W: 4.7 Ω, RC2512FK-074R7L:RC2512FK-074R7L
- added VOLTAGE_REGULATOR: TLV61070A, TLV61070A:TLV61070ASOT-23
- MOSFET2, MOSFET3: value N_CHANNEL -> SSM3K335R; device AO3400A:AO3400A -> SSM3K335R:SSM3K335R
- R2: value 2.7 Ω -> Ω; device RCS08052R70FKEA:RCS08052R70FKEA -> RC0805JR-0720KL:RC0805JR-0720KL
- R5: value 1 kΩ -> Ω
Connections:
- removed net N$16: R2.1, WHITE_LED.2
- new net N$10: L1.2, VOLTAGE_REGULATOR.SW
- new net N$7: R1_1W.1, WHITE_LED1.P
- new net VBAT1: C6.1
- new net VCHARGE: BATTERY_CHARGER.VDD, C1.1, CHARGER_PORT1.P, D1.A
- net 12V: now also ACTIVE_BUZZER1.P, INVERTER.VDD; no longer ACTIVE_BUZZER.2
- net 5V: now also R1_1W.2, R2.2, VOLTAGE_REGULATOR.VOUT; no longer BATTERY_CHARGER.VDD, C1.1, CHARGER_PORT.2, D1.A
- net GND: now also BATTERY2.P, C5.2, C6.2, CHARGER_PORT2.P, INVERTER.VSS, MOSFET2.2, MOSFET3.2, R5.1, VOLTAGE_REGULATOR.GND; no longer BATTERY.1, CHARGER_PORT.1, MOSFET2.S, MOSFET3.S, TRANSISTOR1.E
- net N$11: now also INVERTER.A; no longer R5.1
- net N$12: now also R2.1, VOLTAGE_REGULATOR.FB; no longer TRANSISTOR1.B
- net N$13: now also INVERTER.Y; no longer R8.1, TRANSISTOR1.C
- net N$14: now also MOSFET3.1; no longer MOSFET3.G
- net N$15: now also MOSFET3.3, WHITE_LED2.P; no longer MOSFET3.D, WHITE_LED.1
- net N$18: now also MOSFET2.1; no longer MOSFET2.G
- net N$19: now also ACTIVE_BUZZER2.P, MOSFET2.3; no longer ACTIVE_BUZZER.1, MOSFET2.D
- net VBAT: now also BATTERY1.P, C5.1, L1.1, VOLTAGE_REGULATOR.VIN; no longer BATTERY.2, R2.2, R8.2
- net VIN: now also VOLTAGE_REGULATOR.EN
Other:
- moved on the sheet: 555_TIMER, BOOST_CONVERTER, C3, C4, R2, R5, R6, R7, RA, RB

Commit message: sent for manufacturing
Parts:
- removed C5, C6: GRT21BR61H475ME13L, GRT21BR61H475ME13L:GRT21BR61H475ME13L
- removed R6, R7: 10 Ω, RC0805JR-0720KL:RC0805JR-0720KL
- added CIN, COUT: 4.7 uF, GRT21BR61H475ME13L:GRT21BR61H475ME13L
- added R_LED: 220 Ω, RC0805JR-0720KL:RC0805JR-0720KL
- added R_PROG: 10 kΩ, RC0805JR-0720KL:RC0805JR-0720KL
- added TEST_12V, TEST_555, TEST_5V, TEST_GND, TEST_INVERTER, TEST_VBAT: WIREPADSMD1,27-254, wirepad:WIREPADSMD1,27-254
- 5V_REGULATOR: value TLV61070A -> TLV61070ASOT-23
- C1, C2: value 4.7 uF -> GRT21BR61H475ME13L
- MOSFET_P: value P_CHANNEL -> DMP2004K
- R1: value 10 kΩ -> Ω
- R3: value 220 Ω -> 20 kΩ
- R4: value 20 kΩ -> 10 Ω
- R5: value Ω -> 10 Ω
- REED_SWITCH: value NORMALLY_OPEN -> REED_SWITCH-PTH-GLASS; device SparkFun-Switches:REED_SWITCH-PTH-GLASS -> RI-80GP0510:REED_SWITCH-PTH-GLASS
- renumbered ACTIVE_BUZZER1 to BUZZER_A, ACTIVE_BUZZER2 to BUZZER_C, BATTERY1 to BATTERY_V, BATTERY2 to BAT_GND, BATTERY_CHARGER to CHARGER, BOOST_CONVERTER to 12V_REGULATOR, CHARGER_PORT1 to CHARGER_V, CHARGER_PORT2 to CH_GND, D1 to CHARGER_LED, MOSFET1 to MOSFET_P, MOSFET2 to MOSFET_N1, MOSFET3 to MOSFET_N2, R1_1W to R_1W, VOLTAGE_REGULATOR to 5V_REGULATOR, WHITE_LED1 to LED_A, WHITE_LED2 to LED_C
Connections:
- removed net VBAT1: C6.1
- net 12V: now also TEST_12V.P
- net 5V: now also C2.1, R1.2, TEST_5V.P; no longer R2.2
- net GND: now also CIN.2, COUT.2, R2.1, R3.2, R_PROG.1, TEST_GND.P; no longer C5.2, C6.2, R1.1, R4.2, R5.1
- net N$11: now also TEST_555.P
- net N$12: now also R1.1, R2.2; no longer R2.1, R5.2
- net N$13: now also R4.1, R5.1, TEST_INVERTER.P; no longer R6.1, R7.1
- net N$14: now also R4.2; no longer R7.2
- net N$18: now also R5.2; no longer R6.2
- net N$2: now also R_PROG.2; no longer R1.2
- net N$3: now also R_LED.1; no longer R3.1
- net N$4: now also R3.1; no longer R4.1
- net N$5: now also R_LED.2; no longer R3.2
- net VBAT: now also COUT.1; no longer 5V_REGULATOR.VIN, C2.1, C5.1, L1.1
- net VCHARGE: now also CIN.1; no longer C1.1
- net VIN: now also 5V_REGULATOR.VIN, C1.1, L1.1, TEST_VBAT.P
Other:
- moved on the sheet: C1, C2, R1, R2, R3, R4, R5
